File: MesquiteRX.kicad_pcb (KiCad board)
At the start: 2 copper layers, 28.5 x 43.5 mm, 7 parts, among them J1 Conn_01x02, J10 Conn_Coaxial, U1 RFM95W-915S2, U2 NodeMCU1.0(ESP-12E)

Commit message: Testing Online
MesquiteRX.kicad_pcb: Manufacturing: tenting front back → -; covering -
  → -; plugging - → -; capping - → no; filling - → no; changed the plot
  output settings. Marco Fissore: moved REF**; rerouted CLK, CS, MISO,
  MOSI and 5 more nets.
MesquiteRX.kicad_pro: Manufacturing: changed the IPC-2581 settings.
  Changed outside PCBJam editing: changed teardrop settings; changed
  default text and line settings; changed 6 DRC rule severities; changed
  net class Default; changed schematic settings; changed 1 component
  class settings.assignments setting; changed 1 component class
  settings.meta setting; and 3 more changes.
MesquiteRX.kicad_sch: Marco Fissore rearranged the sheet.
pcbjam.lock.json: Library lockfile regenerated.

Checks: ERC: 49 errors, 1 warning in MesquiteRX.kicad_sch (pin not connected ×24, pin not driven ×21, power pin not driven ×4) · DRC: 14 warnings, 2 unrouted connections in MesquiteRX.kicad_pcb (silk over copper ×9, silk edge clearance ×5)

PCBJam-Commit: 8686b0dd-4d75-4811-8bda-9c8a46edee61
Parts:
- moved REF** 0.50 mm to (136.8, 65.5)
